Commit message: fixed orientation to fit body frame

File: sbr_description/robot.urdf (robot description, URDF)
Before this commit: robot sbr_description, 4 links, 3 joints
Joints:
- joint left_wheel_joint: origin xyz=0.0265233 0.00796397 -0.0669234 rpy=-1.5708 6.12323e-17 1.5708 -> xyz=-7.50005e-05 0.06305 -0.0376433 rpy=-1.5708 6.12323e-17 3.14159
- joint right_wheel_joint: origin xyz=-0.100577 0.00796397 -0.0669234 rpy=-1.5708 -6.12323e-17 -1.5708 -> xyz=-7.50005e-05 -0.06405 -0.0376433 rpy=-1.5708 -6.12323e-17 0
